Commit message: Indentacion, ajuste de multirobot.py, algunos comentarios, etc

File: urdf/pioneer3dx_wheel.xacro (robot description, xacro)
@@ -18,5 +18,5 @@
 <robot xmlns:xacro="http://ros.org/wiki/xacro">
 	<!-- properties (constants) -->
-	<property name="M_PI" value="3.14159" />
+	<xacro:property name="M_PI" value="3.14159" />
 	<!-- right/left hubcap + wheel -->
 	<xacro:macro name="p3dx_wheel" params="suffix parent reflect">
